Commit message: Inertial_commit

File: description/robot_core.xacro (robot description, xacro)
@@ -1,36 +1,119 @@
 <?xml version="1.0"?>
-<robot xmlns:xacro="http://www.ros.org/wiki/xacro" name="robot">
-  <!-- Materials -->
-  <material name="white"><color rgba="1 1 1 1"/></material>
-  <material name="orange"><color rgba="1 0.5 0 1"/></material>
-  <material name="blue"><color rgba="0 0 1 1"/></material>
-  <material name="black"><color rgba="0 0 0 1"/></material>
-  <!-- Chassis dimensions -->
-  <xacro:property name="chassis_L" value="0.275"/>
-  <xacro:property name="chassis_W" value="0.15"/>
-  <xacro:property name="chassis_H" value="0.1"/>
-  <link name="base_link"/>
-  <!-- Chassis frame -->
-  <joint name="chassis_joint" type="fixed">
-    <parent link="base_link"/>
-    <child link="chassis"/>
-    <origin xyz="-0.075 0 0" rpy="0 0 0"/>
-  </joint>
-  <link name="chassis">
-    <visual>
-      <!-- Box origin at the back of AGV -->
-      <origin xyz="${chassis_L/2} 0 ${chassis_H/2}" rpy="0 0 0"/>
-      <geometry>
-        <box size="${chassis_L} ${chassis_W} ${chassis_H}"/>
-      </geometry>
-      <material name="white"/>
-    </visual>
-    <!-- Nên thêm collision giống visual để sau này mô phỏng/plan -->
-    <collision>
-      <origin xyz="${chassis_L/2} 0 ${chassis_H/2}" rpy="0 0 0"/>
-      <geometry>
-        <box size="${chassis_L} ${chassis_W} ${chassis_H}"/>
-      </geometry>
-    </collision>
-  </link>
+<robot xmlns:xacro="http://www.ros.org/wiki/xacro">
+    <!-- Materials -->
+    <material name="white">
+        <color rgba="1 1 1 1"/>
+    </material>
+    <material name="orange">
+        <color rgba="1 0.5 0 1"/>
+    </material>
+    <material name="blue">
+        <color rgba="0 0 1 1"/>
+    </material>
+    <material name="black">
+        <color rgba="0 0 0 1"/>
+    </material>
+    <!-- Chassis dimensions -->
+    <xacro:property name="chassis_L" value="0.275"/>
+    <xacro:property name="chassis_W" value="0.15"/>
+    <xacro:property name="chassis_H" value="0.1"/>
+    <!-- Wheel params -->
+    <xacro:property name="wheel_radius" value="0.037"/>
+    <!-- 74mm diameter -->
+    <xacro:property name="wheel_width" value="0.02"/>
+    <!-- 20mm thick -->
+    <!-- Caster wheel params -->
+    <xacro:property name="caster_radius" value="0.02"/>
+    <!-- Base link -->
+    <link name="base_link">
+    </link>
+    <!-- Chassis frame -->
+    <joint name="chassis_joint" type="fixed">
+        <parent link="base_link"/>
+        <child link="chassis"/>
+        <origin xyz="-0.075 0 0" rpy="0 0 0"/>
+    </joint>
+    <link name="chassis">
+        <visual>
+            <!-- Box origin at the back of AGV -->
+            <origin xyz="${chassis_L/2} 0 ${chassis_H/2}" rpy="0 0 0"/>
+            <geometry>
+                <box size="${chassis_L} ${chassis_W} ${chassis_H}"/>
+            </geometry>
+            <material name="white"/>
+        </visual>
+        <collision>
+            <origin xyz="${chassis_L/2} 0 ${chassis_H/2}" rpy="0 0 0"/>
+            <geometry>
+                <box size="${chassis_L} ${chassis_W} ${chassis_H}"/>
+            </geometry>
+        </collision>
+    </link>
+    <!-- Left wheel -->
+    <joint name="left_wheel_joint" type="continuous">
+        <parent link="base_link"/>
+        <child link="left_wheel"/>
+        <origin xyz="0 ${chassis_W/2 + wheel_width/2} 0" rpy="-${pi/2} 0 0"/>
+        <axis xyz="0 0 1"/>
+    </joint>
+    <link name="left_wheel">
+        <visual>
+            <origin xyz="0 0 0" rpy="0 0 0"/>
+            <geometry>
+                <cylinder length="${wheel_width}" radius="${wheel_radius}"/>
+            </geometry>
+            <material name="black"/>
+        </visual>
+        <collision>
+            <origin xyz="0 0 0" rpy="0 0 0"/>
+            <geometry>
+                <cylinder length="${wheel_width}" radius="${wheel_radius}"/>
+            </geometry>
+        </collision>
+    </link>
+    <!-- Right wheel -->
+    <joint name="right_wheel_joint" type="continuous">
+        <parent link="base_link"/>
+        <child link="right_wheel"/>
+        <origin xyz="0 -${chassis_W/2 + wheel_width/2} 0" rpy="${pi/2} 0 0"/>
+        <axis xyz="0 0 -1"/>
+    </joint>
+    <link name="right_wheel">
+        <visual>
+            <origin xyz="0 0 0" rpy="0 0 0"/>
+            <geometry>
+                <cylinder length="${wheel_width}" radius="${wheel_radius}"/>
+            </geometry>
+            <material name="black"/>
+        </visual>
+        <collision>
+            <origin xyz="0 0 0" rpy="0 0 0"/>
+            <geometry>
+                <cylinder length="${wheel_width}" radius="${wheel_radius}"/>
+            </geometry>
+        </collision>
+    </link>
+    <!-- Caster wheel -->
+    <!-- Caster wheel -->
+    <joint name="caster_wheel_joint" type="fixed">
+        <parent link="chassis"/>
+        <child link="caster_wheel"/>
+        <!-- z = -wheel_radius + caster_radius = -0.037 + 0.02 = -0.017 -->
+        <origin xyz="0.2 0 ${-wheel_radius + caster_radius}" rpy="0 0 0"/>
+    </joint>
+    <link name="caster_wheel">
+        <visual>
+            <origin xyz="0 0 0" rpy="0 0 0"/>
+            <geometry>
+                <sphere radius="${caster_radius}"/>
+            </geometry>
+            <material name="blue"/>
+        </visual>
+        <collision>
+            <origin xyz="0 0 0" rpy="0 0 0"/>
+            <geometry>
+                <sphere radius="${caster_radius}"/>
+            </geometry>
+        </collision>
+    </link>
 </robot>

Commit message: Complete 3D model

File: description/robot_core.xacro (robot description, xacro)
@@ -1,4 +1,5 @@
 <?xml version="1.0"?>
 <robot xmlns:xacro="http://www.ros.org/wiki/xacro">
+    <xacro:include filename="inertial_macros.xacro"/>
     <!-- Materials -->
     <material name="white">
@@ -49,4 +50,7 @@
             </geometry>
         </collision>
+        <xacro:inertial_box mass="0.5" x="${chassis_L}" y="${chassis_W}" z="${chassis_H}">
+            <origin xyz="${chassis_L/2} 0 ${chassis_H/2}" rpy="0 0 0"/>
+        </xacro:inertial_box>
     </link>
     <!-- Left wheel -->
@@ -71,4 +75,7 @@
             </geometry>
         </collision>
+        <xacro:inertial_cylinder mass="0.1" length="${wheel_width}" radius="${wheel_radius}">
+            <origin xyz="0 0 0" rpy="0 0 0"/>
+        </xacro:inertial_cylinder>
     </link>
     <!-- Right wheel -->
@@ -93,6 +100,8 @@
             </geometry>
         </collision>
+        <xacro:inertial_cylinder mass="0.1" length="${wheel_width}" radius="${wheel_radius}">
+            <origin xyz="0 0 0" rpy="0 0 0"/>
+        </xacro:inertial_cylinder>
     </link>
-    <!-- Caster wheel -->
     <!-- Caster wheel -->
     <joint name="caster_wheel_joint" type="fixed">
@@ -116,4 +125,7 @@
             </geometry>
         </collision>
+        <xacro:inertial_sphere mass="0.1" radius="${caster_radius}">
+            <origin xyz="0 0 0" rpy="0 0 0"/>
+        </xacro:inertial_sphere>
     </link>
 </robot>

Commit message: update AGV On Gazbo

File: description/robot_core.xacro (robot description, xacro)
@@ -54,4 +54,7 @@
         </xacro:inertial_box>
     </link>
+    <gazebo reference="chassis">
+        <material>Gazebo/White</material>
+    </gazebo>
     <!-- Left wheel -->
     <joint name="left_wheel_joint" type="continuous">
@@ -79,4 +82,7 @@
         </xacro:inertial_cylinder>
     </link>
+    <gazebo reference="left_wheel">
+        <material>Gazebo/Black</material>
+    </gazebo>
     <!-- Right wheel -->
     <joint name="right_wheel_joint" type="continuous">
@@ -104,4 +110,7 @@
         </xacro:inertial_cylinder>
     </link>
+    <gazebo reference="right_wheel">
+        <material>Gazebo/Black</material>
+    </gazebo>
     <!-- Caster wheel -->
     <joint name="caster_wheel_joint" type="fixed">
@@ -129,3 +138,6 @@
         </xacro:inertial_sphere>
     </link>
+    <gazebo reference="caster_wheel">
+        <material>Gazebo/Blue</material>
+    </gazebo>
 </robot>
