Commit message: update gazebo anh rviz

File: description/gazebo_control.xacro (robot description, xacro)
@@ -1,3 +1,22 @@
 <?xml version="1.0"?>
 <robot xmlns:xacro="http://www.ros.org/wiki/xacro">
+<xacro:include filename="robot_parameters.xacro"/>
+    <gazebo>
+        <plugin name="diff_drive" filename="libgazebo_ros_diff_drive.so">
+            <!--Wheel info-->
+            <left_joint>left_wheel_joint</left_joint>
+            <right_joint>right_wheel_joint</right_joint>
+            <wheel_separation>${chassis_W + wheel_width}</wheel_separation>
+            <wheel_diameter>${wheel_radius*2}</wheel_diameter>
+            <!--Limits-->
+            <max_wheel_torque>200.0</max_wheel_torque>
+            <max_acceleration>10.0</max_acceleration>
+            <!--Output-->
+            <odometry_frame>odom</odometry_frame>
+            <robot_base_frame>base_link</robot_base_frame>
+            <publish_odom>true</publish_odom>
+            <publish_odom_tf>true</publish_odom_tf>
+            <publish_wheel_tf>true</publish_wheel_tf>
+        </plugin>
+    </gazebo>
 </robot>

File: description/robot_core.xacro (robot description, xacro)
@@ -1,4 +1,5 @@
 <?xml version="1.0"?>
 <robot xmlns:xacro="http://www.ros.org/wiki/xacro">
+    <xacro:include filename="robot_parameters.xacro"/>
     <xacro:include filename="inertial_macros.xacro"/>
     <!-- Materials -->
@@ -15,15 +16,4 @@
         <color rgba="0 0 0 1"/>
     </material>
-    <!-- Chassis dimensions -->
-    <xacro:property name="chassis_L" value="0.275"/>
-    <xacro:property name="chassis_W" value="0.15"/>
-    <xacro:property name="chassis_H" value="0.1"/>
-    <!-- Wheel params -->
-    <xacro:property name="wheel_radius" value="0.037"/>
-    <!-- 74mm diameter -->
-    <xacro:property name="wheel_width" value="0.02"/>
-    <!-- 20mm thick -->
-    <!-- Caster wheel params -->
-    <xacro:property name="caster_radius" value="0.02"/>
     <!-- Base link -->
     <link name="base_link">
@@ -140,4 +130,6 @@
     <gazebo reference="caster_wheel">
         <material>Gazebo/Blue</material>
+        <mu1 value="0.001"/>
+        <mu2 value="0.001"/>
     </gazebo>
 </robot>
